File: VolvocineWithCurrentSensorV4.kicad_pcb (KiCad board)
At the start: 2 copper layers, 29 x 32.3 mm, 30 parts, among them J2 Conn_01x12_Socket, J3 Sensors, J4 Switch, J5 battery, J6 Conn_01x12_Socket, Q2 Si2315, U1 PAM2401SCADJ, U2 PIC10F322-IOT, U3 INA226

Commit message: Autosave
Parts:
- RFB1: value 750k -> 330k
Changed lines of the file:
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@@
 			)
 		)
-		(property "Value" "750k"
+		(property "Value" "330k"
 			(at 0.07825 -1.057 0)
 			(layer "F.Fab")

Commit message: Autosave
Parts:
- RFB2: value 100k -> 47k
Changed lines of the file:
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@@
 			)
 		)
-		(property "Value" "100k"
+		(property "Value" "47k"
 			(at 0.03125 -1.057 0)
 			(layer "F.Fab")
